Commit message: URDF changed so the start state wouldn't be in collision.

File: robotnik_powerball_description/urdf/powerball_gripper.urdf (robot description, URDF)
Before this commit: robot powerball, 14 links, 13 joints
Joints:
- joint base_joint_gripper_left: limit lower=-0.055 upper=-0.0027 effort=1.0 velocity=1.0 -> lower=-0.055 upper=-0.004 effort=1.0 velocity=1.0
- joint base_joint_gripper_right: limit lower=0.0027 upper=0.055 effort=1.0 velocity=1.0 -> lower=0.004 upper=0.055 effort=1.0 velocity=1.0
- joint guide_joint_finger_left: origin xyz=0 0 0.023 rpy=0 0 0 -> xyz=0 0 0.024 rpy=0 0 0
- joint guide_joint_finger_right: origin xyz=0 0 0.023 rpy=0 0 0 -> xyz=0 0 0.024 rpy=0 0 0

Commit message: Base visual and friction changed because of slipping.
Will need to play with the coefficients, because it
still slips.

File: robotnik_powerball_description/urdf/powerball_gripper.urdf (robot description, URDF)
Before this commit: robot powerball, 14 links, 13 joints
Links:
- link base_link: geometry collision box size=0.2 0.3 0.5; visual box size=0.2 0.3 0.5

Commit message: Joint limits edited (planning more successful).
Removed some parts of the URDF, e.g. tool_link.

File: robotnik_powerball_description/urdf/powerball_gripper.urdf (robot description, URDF)
Before this commit: robot powerball, 14 links, 13 joints
Links:
- removed link tool_link
Joints:
- removed joint gripper_base_link_tool_joint
- joint arm_1_joint: limit lower=-2.97 upper=2.97 effort=370 velocity=2.0 -> lower=-3.1416 upper=3.1416 effort=370 velocity=2.0
- joint arm_2_joint: limit lower=-1.92 upper=1.92 effort=370 velocity=2.0 -> lower=-3.1416 upper=3.1416 effort=370 velocity=2.0
- joint arm_3_joint: limit lower=-2.71 upper=2.71 effort=176 velocity=2.0 -> lower=-3.1416 upper=3.1416 effort=176 velocity=2.0
- joint arm_4_joint: limit lower=-2.97 upper=2.97 effort=176 velocity=2.0 -> lower=-3.1416 upper=3.1416 effort=176 velocity=2.0
- joint arm_5_joint: limit lower=-2.44 upper=2.44 effort=41.6 velocity=2.0 -> lower=-3.1416 upper=3.1416 effort=41.6 velocity=2.0
- joint arm_6_joint: limit lower=-2.97 upper=2.97 effort=20.1 velocity=2.0 -> lower=-3.1416 upper=3.1416 effort=20.1 velocity=2.0

Commit message: Correct joint limits entered...
...except for the soft limit on joint 3.

File: robotnik_powerball_description/urdf/powerball_gripper.urdf (robot description, URDF)
Before this commit: robot powerball, 13 links, 12 joints
Joints:
- joint arm_1_joint: limit lower=-3.1416 upper=3.1416 effort=370 velocity=2.0 -> lower=-2.9671 upper=2.9671 effort=370 velocity=2.0
- joint arm_2_joint: limit lower=-3.1416 upper=3.1416 effort=370 velocity=2.0 -> lower=-2.9671 upper=2.9671 effort=370 velocity=2.0
- joint arm_3_joint: limit lower=-3.1416 upper=3.1416 effort=176 velocity=2.0 -> lower=-2.9671 upper=2.9671 effort=176 velocity=2.0
- joint arm_4_joint: limit lower=-3.1416 upper=3.1416 effort=176 velocity=2.0 -> lower=-2.9671 upper=2.9671 effort=176 velocity=2.0
- joint arm_5_joint: limit lower=-3.1416 upper=3.1416 effort=41.6 velocity=2.0 -> lower=-2.9671 upper=2.9671 effort=41.6 velocity=2.0
- joint arm_6_joint: limit lower=-3.1416 upper=3.1416 effort=20.1 velocity=2.0 -> lower=-2.9671 upper=2.9671 effort=20.1 velocity=2.0
